File: RF AMP 1W.brd (EAGLE design)
At the start: 100 x 66 mm, 40 parts, among them Q1 BFY50, Q3 BFY50, T1 BUX85

Commit message: fixed missing net, trace width 1mm
Connections:
- new net N$17: L3.OUT1, T1.1
- net N$18: now also L3.OUT2
Routing:
- net N$18: track 40.0 -> 65.2 mm
- net N$17: track 0.00 -> 17.6 mm
